File: HOBE/HOBE.kicad_sch (KiCad schematic)
At the start: 0 parts

Commit message: pretty
Other:
- company: (none) -> EE198
- title: (none) -> HOPE Final Project

Commit message: stuff
Parts:
- added IC1: TESEO-LIV3F, SON110P970X1010X230-18N, symbol HOPE_Footprint:TESEO-LIV3F
- added IC2: PAM8403DR, SOIC127P600X126-16N, symbol HOPE_Footprint:PAM8403DR
- added MK1: ICS-43434, ICS-43434:MIC_ICS-43434, symbol HOPE_Footprint:ICS-43434
- added U1: LSM6DSVTR, LGA14-L_2P59X3P1X0P5_STM, symbol HOPE_Footprint:LSM6DSVTR
- added U2: STM32WL33CCV6, VFQFPN-48_6x6x0p9mm_STM, symbol HOPE_Footprint:STM32WL33CCV6
